Commit message: feat(motion): 验证抽离后负重姿态规划
- 将 v5 link3 关节段加长 0.1m，并更新抽离 benchmark 的负重姿态。

- 增加抽离成功后到 dual_v5_arm 负重姿态的 MoveIt 规划验证。

- 记录负重规划成功率、耗时、轨迹点数和附着箱碰撞失败原因。

Co-Authored-By: Codex <codex@openai.com>

Refs MOTION-51

File: ros2_ws/src/alfa_robot_description/urdf/alfa_robot.urdf.xacro (robot description, xacro)
@@ -248,5 +248,5 @@
   </link>
 <joint name="left_v5_joint4" type="revolute">
-    <origin xyz="0.0010609 -0.239 -0.077993" rpy="1.5708 0 0" />
+    <origin xyz="0.0010609 -0.339 -0.077993" rpy="1.5708 0 0" />
     <parent link="left_v5_link3" />
     <child link="left_v5_link4" />
@@ -447,5 +447,5 @@
   </link>
 <joint name="right_v5_joint4" type="revolute">
-    <origin xyz="-0.0010609 -0.239 0.077993" rpy="1.5708 0 0" />
+    <origin xyz="-0.0010609 -0.339 0.077993" rpy="1.5708 0 0" />
     <parent link="right_v5_link3" />
     <child link="right_v5_link4" />

Commit message: feat(motion): 迁移新机械臂初版模型
- 迁入 v9 机械臂 visual/collision mesh 资产，并切换 URDF 关节原点、惯量和 mesh 引用。
- 同步 ros2_control、MoveIt SRDF、初始姿态、关节限制和 MuJoCo 初始姿态配置。
- 保留既有 left_v5/right_v5/tool0 对外接口名，记录后续 TCP 与自碰撞矩阵复核风险。

验证：
- xacro + check_urdf 通过 description 与 MoveIt wrapper。
- colcon build --packages-select alfa_robot_description alfa_robot_moveit_config --symlink-install --cmake-args -DBUILD_TESTING=OFF 通过。

Co-Authored-By: Codex <codex@openai.com>

Refs MOTION-59

File: ros2_ws/src/alfa_robot_description/urdf/alfa_robot.urdf.xacro (robot description, xacro)
@@ -17,49 +17,577 @@
     <origin xyz="0 0 0.202094" rpy="0 0 0"/>
   </joint>
-<link name="base_link">
-    <inertial>
-      <origin xyz="-0.230864859994365 -3.59465059753261E-05 0.00982453569098829" rpy="0 0 0" />
-      <mass value="452.254374649793" />
-      <inertia ixx="42.2528118012676" ixy="2.90433873726581E-05" ixz="5.29862244779797" iyy="45.7334828734001" iyz="-7.53976926824646E-07" izz="73.6321595788915" />
-    </inertial>
-    <visual>
-      <origin xyz="0 0 0" rpy="0 0 0" />
-      <geometry>
-        <mesh filename="package://alfa_robot_description/meshes/alfa_robot_v2_arm_v6/visual/base_link.STL" />
-      </geometry>
-      <material name="">
-        <color rgba="0.752941176470588 0.752941176470588 0.752941176470588 1" />
-      </material>
-    </visual>
-    <collision>
-      <origin xyz="0 0 0" rpy="0 0 0" />
-      <geometry>
-        <mesh filename="package://alfa_robot_description/meshes/alfa_robot_v2_arm_v6/collision/base_link.STL" />
-      </geometry>
-    </collision>
-  </link>
-<link name="pitch">
-    <inertial>
-      <origin xyz="-0.197037068600063 0.0545002757388739 0.0847212210627051" rpy="0 0 0" />
-      <mass value="31.6067905352622" />
-      <inertia ixx="0.518725062034511" ixy="2.02803901410849E-08" ixz="-0.00603915225902053" iyy="0.579528262067602" iyz="3.22538967579058E-07" izz="1.06221345040969" />
-    </inertial>
-    <visual>
-      <origin xyz="0 0 0" rpy="0 0 0" />
-      <geometry>
-        <mesh filename="package://alfa_robot_description/meshes/alfa_robot_v2_arm_v6/visual/pitch.STL" />
-      </geometry>
-      <material name="">
-        <color rgba="0.752941176470588 0.752941176470588 0.752941176470588 1" />
-      </material>
-    </visual>
-    <collision>
-      <origin xyz="0 0 0" rpy="0 0 0" />
-      <geometry>
-        <mesh filename="package://alfa_robot_description/meshes/alfa_robot_v2_arm_v6/collision/pitch.STL" />
-      </geometry>
-    </collision>
-  </link>
-<joint name="pitch" type="revolute">
+  <link name="base_link">
+    <inertial>
+      <origin xyz="-0.23088491629759 -3.59403635409317E-05 0.0098300335923529" rpy="0 0 0" />
+      <mass value="452.331665683053" />
+      <inertia ixx="42.2528214496965" ixy="2.9043387371881E-05" ixz="5.29862244779798" iyy="45.7349589120892" iyz="-7.53976926755255E-07" izz="73.6336356175806" />
+    </inertial>
+    <visual>
+      <origin xyz="0 0 0" rpy="0 0 0" />
+      <geometry>
+        <mesh filename="package://alfa_robot_description/meshes/alfa_robot_v2_arm_v9/visual/base_link.STL" />
+      </geometry>
+      <material name="">
+        <color rgba="0.752941176470588 0.752941176470588 0.752941176470588 1" />
+      </material>
+    </visual>
+    <collision>
+      <origin xyz="0 0 0" rpy="0 0 0" />
+      <geometry>
+        <mesh filename="package://alfa_robot_description/meshes/alfa_robot_v2_arm_v9/collision/base_link.STL" />
+      </geometry>
+    </collision>
+  </link>
+  <link name="pitch">
+    <inertial>
+      <origin xyz="-0.197223755735604 0.0545002751304143 0.0848583683408157" rpy="0 0 0" />
+      <mass value="31.6766900042973" />
+      <inertia ixx="0.518885879634885" ixy="2.02803902279695E-08" ixz="-0.00591642486892729" iyy="0.580169083875299" iyz="3.22538967431134E-07" izz="1.06295541093974" />
+    </inertial>
+    <visual>
+      <origin xyz="0 0 0" rpy="0 0 0" />
+      <geometry>
+        <mesh filename="package://alfa_robot_description/meshes/alfa_robot_v2_arm_v9/visual/pitch.STL" />
+      </geometry>
+      <material name="">
+        <color rgba="0.752941176470588 0.752941176470588 0.752941176470588 1" />
+      </material>
+    </visual>
+    <collision>
+      <origin xyz="0 0 0" rpy="0 0 0" />
+      <geometry>
+        <mesh filename="package://alfa_robot_description/meshes/alfa_robot_v2_arm_v9/collision/pitch.STL" />
+      </geometry>
+    </collision>
+  </link>
+  <link name="turn">
+    <inertial>
+      <origin xyz="-0.00958110945289126 -7.73859721442394E-06 1.06018839944043" rpy="0 0 0" />
+      <mass value="53.4681885650186" />
+      <inertia ixx="7.9404350019494" ixy="5.99860879545119E-06" ixz="0.185339515626497" iyy="8.17240800709107" iyz="-8.94803411816649E-06" izz="0.75519185821394" />
+    </inertial>
+    <visual>
+      <origin xyz="0 0 0" rpy="0 0 0" />
+      <geometry>
+        <mesh filename="package://alfa_robot_description/meshes/alfa_robot_v2_arm_v9/visual/turn.STL" />
+      </geometry>
+      <material name="">
+        <color rgba="0.752941176470588 0.752941176470588 0.752941176470588 1" />
+      </material>
+    </visual>
+    <collision>
+      <origin xyz="0 0 0" rpy="0 0 0" />
+      <geometry>
+        <mesh filename="package://alfa_robot_description/meshes/alfa_robot_v2_arm_v9/collision/turn.STL" />
+      </geometry>
+    </collision>
+  </link>
+  <link name="updown">
+    <inertial>
+      <origin xyz="0.0637333774739139 -2.9260470713055E-09 0.104211014753683" rpy="0 0 0" />
+      <mass value="24.4167257440598" />
+      <inertia ixx="1.07967195604977" ixy="-1.55435028024514E-08" ixz="-0.00582099906204064" iyy="0.231957862842844" iyz="9.04966240965367E-11" izz="1.26737556353379" />
+    </inertial>
+    <visual>
+      <origin xyz="0 0 0" rpy="0 0 0" />
+      <geometry>
+        <mesh filename="package://alfa_robot_description/meshes/alfa_robot_v2_arm_v9/visual/updown.STL" />
+      </geometry>
+      <material name="">
+        <color rgba="0.752941176470588 0.752941176470588 0.752941176470588 1" />
+      </material>
+    </visual>
+    <collision>
+      <origin xyz="0 0 0" rpy="0 0 0" />
+      <geometry>
+        <mesh filename="package://alfa_robot_description/meshes/alfa_robot_v2_arm_v9/collision/updown.STL" />
+      </geometry>
+    </collision>
+  </link>
+  <!-- ========== LEFT ARM v9 mapped to left_v5_* project names ========== -->
+  <link name="left_v5_link0">
+    <inertial>
+      <origin xyz="0 0 0" rpy="0 0 0"/>
+      <mass value="0.001"/>
+      <inertia ixx="1e-6" ixy="0" ixz="0" iyy="1e-6" iyz="0" izz="1e-6"/>
+    </inertial>
+  </link>
+  <joint name="left_v5_mount" type="fixed">
+    <parent link="updown"/>
+    <child link="left_v5_link0"/>
+    <origin xyz="0.095 0.26 0.2" rpy="0 0 0"/>
+  </joint>
+  <link name="left_v5_link1">
+    <inertial>
+      <origin xyz="1.9813263254731E-05 0.00247298217574687 0.0580356323599454" rpy="0 0 0" />
+      <mass value="2.53849365971103" />
+      <inertia ixx="0.00565316591359282" ixy="1.39299660407887E-06" ixz="-2.78630772083778E-06" iyy="0.00554455173094211" iyz="-7.0690628326149E-05" izz="0.00447417412424851" />
+    </inertial>
+    <visual>
+      <origin xyz="0 0 0" rpy="0 0 0" />
+      <geometry>
+        <mesh filename="package://alfa_robot_description/meshes/alfa_robot_v2_arm_v9/visual/leftjoint1.STL" />
+      </geometry>
+      <material name="">
+        <color rgba="0.752941176470588 0.752941176470588 0.752941176470588 1" />
+      </material>
+    </visual>
+    <collision>
+      <origin xyz="0 0 0" rpy="0 0 0" />
+      <geometry>
+        <mesh filename="package://alfa_robot_description/meshes/alfa_robot_v2_arm_v9/collision/leftjoint1.STL" />
+      </geometry>
+    </collision>
+  </link>
+  <joint name="left_v5_joint1" type="revolute">
+    <origin xyz="0 0 0" rpy="0 0 0" />
+    <parent link="left_v5_link0" />
+    <child link="left_v5_link1" />
+    <axis xyz="0 0 1" />
+    <limit lower="-2.35619449" upper="2.35619449" effort="120" velocity="1.2" />
+  </joint>
+  <link name="left_v5_link2">
+    <inertial>
+      <origin xyz="-3.91993193460394E-09 -0.198242241905549 0.0685963634370443" rpy="0 0 0" />
+      <mass value="13.5734229269593" />
+      <inertia ixx="0.347009291103137" ixy="1.79330552144141E-12" ixz="2.19848829810308E-12" iyy="0.0505989087942829" iyz="4.33554113881788E-12" izz="0.367314390536816" />
+    </inertial>
+    <visual>
+      <origin xyz="0 0 0" rpy="0 0 0" />
+      <geometry>
+        <mesh filename="package://alfa_robot_description/meshes/alfa_robot_v2_arm_v9/visual/leftjoint2.STL" />
+      </geometry>
+      <material name="">
+        <color rgba="0.752941176470588 0.752941176470588 0.752941176470588 1" />
+      </material>
+    </visual>
+    <collision>
+      <origin xyz="0 0 0" rpy="0 0 0" />
+      <geometry>
+        <mesh filename="package://alfa_robot_description/meshes/alfa_robot_v2_arm_v9/collision/leftjoint2.STL" />
+      </geometry>
+    </collision>
+  </link>
+  <joint name="left_v5_joint2" type="revolute">
+    <origin xyz="0 0.0825 0.0579999999999996" rpy="-1.5707963267949 0 0" />
+    <parent link="left_v5_link1" />
+    <child link="left_v5_link2" />
+    <axis xyz="0 0 1" />
+    <limit lower="-3.14159265" upper="3.14159265" effort="120" velocity="1.2" />
+  </joint>
+  <link name="left_v5_link3">
+    <inertial>
+      <origin xyz="4.24816812838458E-08 -0.171995906773402 -0.0220559637033981" rpy="0 0 0" />
+      <mass value="5.37152510221438" />
+      <inertia ixx="0.103379389320522" ixy="1.01375731816284E-08" ixz="4.8440173396198E-09" iyy="0.0137404008500263" iyz="0.000240093301068499" izz="0.114911955120257" />
+    </inertial>
+    <visual>
+      <origin xyz="0 0 0" rpy="0 0 0" />
+      <geometry>
+        <mesh filename="package://alfa_robot_description/meshes/alfa_robot_v2_arm_v9/visual/leftjoint3.STL" />
+      </geometry>
+      <material name="">
+        <color rgba="0.752941176470588 0.752941176470588 0.752941176470588 1" />
+      </material>
+    </visual>
+    <collision>
+      <origin xyz="0 0 0" rpy="0 0 0" />
+      <geometry>
+        <mesh filename="package://alfa_robot_description/meshes/alfa_robot_v2_arm_v9/collision/leftjoint3.STL" />
+      </geometry>
+    </collision>
+  </link>
+  <joint name="left_v5_joint3" type="revolute">
+    <origin xyz="0 -0.4 0.008" rpy="0 0 0" />
+    <parent link="left_v5_link2" />
+    <child link="left_v5_link3" />
+    <axis xyz="0 0 1" />
+    <limit lower="-3.14159265" upper="3.14159265" effort="100" velocity="1.2" />
+  </joint>
+  <link name="left_v5_link4">
+    <inertial>
+      <origin xyz="1.86328980931183E-05 0.00232765205467672 0.0541835839509776" rpy="0 0 0" />
+      <mass value="2.69701889029267" />
+      <inertia ixx="0.00655846785174234" ixy="1.39368136512847E-06" ixz="-2.78625493222266E-06" iyy="0.00644984634538746" iyz="-7.06885588830852E-05" izz="0.00474081047943518" />
+    </inertial>
+    <visual>
+      <origin xyz="0 0 0" rpy="0 0 0" />
+      <geometry>
+        <mesh filename="package://alfa_robot_description/meshes/alfa_robot_v2_arm_v9/visual/leftjoint4.STL" />
+      </geometry>
+      <material name="">
+        <color rgba="0.752941176470588 0.752941176470588 0.752941176470588 1" />
+      </material>
+    </visual>
+    <collision>
+      <origin xyz="0 0 0" rpy="0 0 0" />
+      <geometry>
+        <mesh filename="package://alfa_robot_description/meshes/alfa_robot_v2_arm_v9/collision/leftjoint4.STL" />
+      </geometry>
+    </collision>
+  </link>
+  <joint name="left_v5_joint4" type="revolute">
+    <origin xyz="0 -0.34 0.021" rpy="0 0 3.14159265" />
+    <parent link="left_v5_link3" />
+    <child link="left_v5_link4" />
+    <axis xyz="0 0 1" />
+    <limit lower="-3.14159265" upper="3.14159265" effort="60" velocity="1.5" />
+  </joint>
+  <link name="left_v5_link5">
+    <inertial>
+      <origin xyz="0.00232761885815602 1.86282477868636E-05 -0.0541835932362763" rpy="0 0 0" />
+      <mass value="2.69701788961671" />
+      <inertia ixx="0.00644984661938229" ixy="1.39391456321868E-06" ixz="7.06885192212674E-05" iyy="0.00655846677978978" iyz="2.78593765675197E-06" izz="0.00474081002137946" />
+    </inertial>
+    <visual>
+      <origin xyz="0 0 0" rpy="0 0 0" />
+      <geometry>
+        <mesh filename="package://alfa_robot_description/meshes/alfa_robot_v2_arm_v9/visual/leftjoint5.STL" />
+      </geometry>
+      <material name="">
+        <color rgba="0.752941176470588 0.752941176470588 0.752941176470588 1" />
+      </material>
+    </visual>
+    <collision>
+      <origin xyz="0 0 0" rpy="0 0 0" />
+      <geometry>
+        <mesh filename="package://alfa_robot_description/meshes/alfa_robot_v2_arm_v9/collision/leftjoint5.STL" />
+      </geometry>
+    </collision>
+  </link>
+  <joint name="left_v5_joint5" type="revolute">
+    <origin xyz="0 0.076 0.058" rpy="-1.5708 0 3.14159265" />
+    <parent link="left_v5_link4" />
+    <child link="left_v5_link5" />
+    <axis xyz="0 0 1" />
+    <limit lower="-3.14159265" upper="3.14159265" effort="60" velocity="1.5" />
+  </joint>
+  <link name="left_v5_link6">
+    <inertial>
+      <origin xyz="0.000656912040294833 0.000831354480711873 0.143020209405825" rpy="0 0 0" />
+      <mass value="9.66858880038429" />
+      <inertia ixx="0.0956031747008675" ixy="2.07680535741587E-07" ixz="-3.59179174277101E-07" iyy="0.0736864446539421" iyz="-1.65114179066885E-07" izz="0.104451818743786" />
+    </inertial>
+    <visual>
+      <origin xyz="0 0 0" rpy="0 0 0" />
+      <geometry>
+        <mesh filename="package://alfa_robot_description/meshes/alfa_robot_v2_arm_v9/visual/leftjoint6.STL" />
+      </geometry>
+      <material name="">
+        <color rgba="0.752941176470588 0.752941176470588 0.752941176470588 1" />
+      </material>
+    </visual>
+    <collision>
+      <origin xyz="0 0 0" rpy="0 0 0" />
+      <geometry>
+        <mesh filename="package://alfa_robot_description/meshes/alfa_robot_v2_arm_v9/collision/leftjoint6.STL" />
+      </geometry>
+    </collision>
+  </link>
+  <joint name="left_v5_joint6" type="revolute">
+    <origin xyz="0.0825 0 -0.058" rpy="0 1.5708 0" />
+    <parent link="left_v5_link5" />
+    <child link="left_v5_link6" />
+    <axis xyz="0 0 1" />
+    <limit lower="-3.14159265" upper="3.14159265" effort="40" velocity="1.5" />
+  </joint>
+  <!-- ========== RIGHT ARM v9 mapped to right_v5_* project names ========== -->
+  <link name="right_v5_link0">
+    <inertial>
+      <origin xyz="0 0 0" rpy="0 0 0"/>
+      <mass value="0.001"/>
+      <inertia ixx="1e-6" ixy="0" ixz="0" iyy="1e-6" iyz="0" izz="1e-6"/>
+    </inertial>
+  </link>
+  <joint name="right_v5_mount" type="fixed">
+    <parent link="updown"/>
+    <child link="right_v5_link0"/>
+    <origin xyz="0.095 -0.26 0.2" rpy="0 0 0"/>
+  </joint>
+  <link name="right_v5_link1">
+    <inertial>
+      <origin xyz="-1.97935614576483E-05 -0.00247298310211053 0.0580356306667498" rpy="0 0 0" />
+      <mass value="2.53849328920242" />
+      <inertia ixx="0.00565316574735217" ixy="1.39345995845525E-06" ixz="2.78607721482458E-06" iyy="0.0055445517719625" iyz="7.06907347563799E-05" izz="0.0044741740915532" />
+    </inertial>
+    <visual>
+      <origin xyz="0 0 0" rpy="0 0 0" />
+      <geometry>
+        <mesh filename="package://alfa_robot_description/meshes/alfa_robot_v2_arm_v9/visual/rightjoint1.STL" />
+      </geometry>
+      <material name="">
+        <color rgba="0.752941176470588 0.752941176470588 0.752941176470588 1" />
+      </material>
+    </visual>
+    <collision>
+      <origin xyz="0 0 0" rpy="0 0 0" />
+      <geometry>
+        <mesh filename="package://alfa_robot_description/meshes/alfa_robot_v2_arm_v9/collision/rightjoint1.STL" />
+      </geometry>
+    </collision>
+  </link>
+  <joint name="right_v5_joint1" type="revolute">
+    <origin xyz="0 0 0" rpy="0 0 0" />
+    <parent link="right_v5_link0" />
+    <child link="right_v5_link1" />
+    <axis xyz="0 0 1" />
+    <limit lower="-2.35619449" upper="2.35619449" effort="120" velocity="1.2" />
+  </joint>
+  <link name="right_v5_link2">
+    <inertial>
+      <origin xyz="-3.93094112816073E-09 -0.198242241906286 -0.0685963669555523" rpy="0 0 0" />
+      <mass value="13.573422926924" />
+      <inertia ixx="0.347009291103142" ixy="-1.77065393597298E-12" ixz="2.09998862500701E-12" iyy="0.0505989087942401" iyz="-4.27592519983108E-12" izz="0.367314390536786" />
+    </inertial>
+    <visual>
+      <origin xyz="0 0 0" rpy="0 0 0" />
+      <geometry>
+        <mesh filename="package://alfa_robot_description/meshes/alfa_robot_v2_arm_v9/visual/rightjoint2.STL" />
+      </geometry>
+      <material name="">
+        <color rgba="0.752941176470588 0.752941176470588 0.752941176470588 1" />
+      </material>
+    </visual>
+    <collision>
+      <origin xyz="0 0 0" rpy="0 0 0" />
+      <geometry>
+        <mesh filename="package://alfa_robot_description/meshes/alfa_robot_v2_arm_v9/collision/rightjoint2.STL" />
+      </geometry>
+    </collision>
+  </link>
+  <joint name="right_v5_joint2" type="revolute">
+    <origin xyz="0 -0.0825 0.058" rpy="-1.5708 0 0" />
+    <parent link="right_v5_link1" />
+    <child link="right_v5_link2" />
+    <axis xyz="0 0 1" />
+    <limit lower="-3.14159265" upper="3.14159265" effort="120" velocity="1.2" />
+  </joint>
+  <link name="right_v5_link3">
+    <inertial>
+      <origin xyz="-3.26463309718861E-08 -0.171995918001188 0.0220559616889885" rpy="0 0 0" />
+      <mass value="5.37152403365307" />
+      <inertia ixx="0.103379343597945" ixy="-9.45207764856994E-09" ixz="3.87847492796146E-09" iyy="0.0137404004302148" iyz="-0.000240092285835305" izz="0.114911909588075" />
+    </inertial>
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
File: ros2_ws/src/alfa_robot_description/urdf/alfa_robot/alfa_robot_macro.ros2_control.xacro (robot description, xacro)
@@ -14,16 +14,16 @@
                pitch_initial:=0.0
                turn_initial:=0.0
-               updown_initial:=0.45
+               updown_initial:=0.0
                left_v5_joint1_initial:=0.0
-               left_v5_joint2_initial:=0.26179939
-               left_v5_joint3_initial:=2.35619449
+               left_v5_joint2_initial:=0.0
+               left_v5_joint3_initial:=0.0
                left_v5_joint4_initial:=0.0
-               left_v5_joint5_initial:=1.04719755
+               left_v5_joint5_initial:=0.0
                left_v5_joint6_initial:=0.0
                right_v5_joint1_initial:=0.0
-               right_v5_joint2_initial:=0.26179939
-               right_v5_joint3_initial:=2.35619449
+               right_v5_joint2_initial:=0.0
+               right_v5_joint3_initial:=0.0
                right_v5_joint4_initial:=0.0
-               right_v5_joint5_initial:=1.04719755
+               right_v5_joint5_initial:=0.0
                right_v5_joint6_initial:=0.0"
                >
@@ -81,5 +81,5 @@
         <command_interface name="position">
           <param name="min">0</param>
-          <param name="max">0.99</param>
+          <param name="max">0.92</param>
         </command_interface>
         <state_interface name="position">
@@ -103,15 +103,15 @@
         </joint>
       </xacro:macro>
-      <xacro:v5_proxy_control_joint joint_name="left_v5_joint1" lower="-2.35619449" upper="2.35619449" velocity="1.2" initial_value="${left_v5_joint1_initial}"/>
+      <xacro:v5_proxy_control_joint joint_name="left_v5_joint1" lower="-0.0" upper="0.0" velocity="1.2" initial_value="${left_v5_joint1_initial}"/>
       <xacro:v5_proxy_control_joint joint_name="left_v5_joint2" lower="-3.14159265" upper="3.14159265" velocity="1.2" initial_value="${left_v5_joint2_initial}"/>
       <xacro:v5_proxy_control_joint joint_name="left_v5_joint3" lower="-3.14159265" upper="3.14159265" velocity="1.2" initial_value="${left_v5_joint3_initial}"/>
       <xacro:v5_proxy_control_joint joint_name="left_v5_joint4" lower="-3.14159265" upper="3.14159265" velocity="1.5" initial_value="${left_v5_joint4_initial}"/>
-      <xacro:v5_proxy_control_joint joint_name="left_v5_joint5" lower="-2.53072742" upper="2.53072742" velocity="1.5" initial_value="${left_v5_joint5_initial}"/>
+      <xacro:v5_proxy_control_joint joint_name="left_v5_joint5" lower="-3.14159265" upper="3.14159265" velocity="1.5" initial_value="${left_v5_joint5_initial}"/>
       <xacro:v5_proxy_control_joint joint_name="left_v5_joint6" lower="-3.14159265" upper="3.14159265" velocity="1.5" initial_value="${left_v5_joint6_initial}"/>
-      <xacro:v5_proxy_control_joint joint_name="right_v5_joint1" lower="-2.35619449" upper="2.35619449" velocity="1.2" initial_value="${right_v5_joint1_initial}"/>
+      <xacro:v5_proxy_control_joint joint_name="right_v5_joint1" lower="-0.0" upper="0.0" velocity="1.2" initial_value="${right_v5_joint1_initial}"/>
       <xacro:v5_proxy_control_joint joint_name="right_v5_joint2" lower="-3.14159265" upper="3.14159265" velocity="1.2" initial_value="${right_v5_joint2_initial}"/>
       <xacro:v5_proxy_control_joint joint_name="right_v5_joint3" lower="-3.14159265" upper="3.14159265" velocity="1.2" initial_value="${right_v5_joint3_initial}"/>
       <xacro:v5_proxy_control_joint joint_name="right_v5_joint4" lower="-3.14159265" upper="3.14159265" velocity="1.5" initial_value="${right_v5_joint4_initial}"/>
-      <xacro:v5_proxy_control_joint joint_name="right_v5_joint5" lower="-2.53072742" upper="2.53072742" velocity="1.5" initial_value="${right_v5_joint5_initial}"/>
+      <xacro:v5_proxy_control_joint joint_name="right_v5_joint5" lower="-3.14159265" upper="3.14159265" velocity="1.5" initial_value="${right_v5_joint5_initial}"/>
       <xacro:v5_proxy_control_joint joint_name="right_v5_joint6" lower="-3.14159265" upper="3.14159265" velocity="1.5" initial_value="${right_v5_joint6_initial}"/>
     </ros2_control>
