Commit message: refactor(robot): 收口新机械臂命名与仓库资产
- 将当前机械臂模型收口到 current_robot mesh 和无版本语义的关节、group、controller 命名。
- 同步 description、MoveIt、bringup、execution bridge、scene service、MuJoCo 与 benchmark 脚本中的新命名。
- 移除旧代际 mesh、废弃 URDF 入口、pick_ik/trac_ik 依赖包和旧 IK 安装脚本。
- 更新 IK 服务口径、命名护栏文档和协作日志，保留当前 BioIK/KDL 主线能力。

验证：
- git diff --cached --check 通过。
- colcon build --packages-select alfa_robot_description robot_motion_scene_service alfa_robot_moveit_config alfa_robot_bringup alfa_robot_execution_bridge alfa_robot_benchmarks --symlink-install --cmake-args -DBUILD_TESTING=OFF 通过。
- colcon build --packages-select robot_motion_scene_service alfa_robot_moveit_config --symlink-install --cmake-args -DBUILD_TESTING=ON 通过。
- colcon test --packages-select robot_motion_scene_service alfa_robot_moveit_config --return-code-on-test-failure 通过；colcon test-result --verbose 显示 15 tests, 0 errors, 0 failures。

Co-Authored-By: Codex <codex@openai.com>

File: ros2_ws/src/alfa_robot_description/urdf/alfa_robot.urdf.xacro (robot description, xacro)
@@ -19,21 +19,21 @@
   <link name="base_link">
     <inertial>
-      <origin xyz="-0.23088491629759 -3.59403635409317E-05 0.0098300335923529" rpy="0 0 0" />
+      <origin xyz="-0.230884916297589 -3.59403635404876E-05 0.0098300335923569" rpy="0 0 0" />
       <mass value="452.331665683053" />
-      <inertia ixx="42.2528214496965" ixy="2.9043387371881E-05" ixz="5.29862244779798" iyy="45.7349589120892" iyz="-7.53976926755255E-07" izz="73.6336356175806" />
-    </inertial>
-    <visual>
-      <origin xyz="0 0 0" rpy="0 0 0" />
-      <geometry>
-        <mesh filename="package://alfa_robot_description/meshes/alfa_robot_v2_arm_v9/visual/base_link.STL" />
-      </geometry>
-      <material name="">
-        <color rgba="0.752941176470588 0.752941176470588 0.752941176470588 1" />
-      </material>
-    </visual>
-    <collision>
-      <origin xyz="0 0 0" rpy="0 0 0" />
-      <geometry>
-        <mesh filename="package://alfa_robot_description/meshes/alfa_robot_v2_arm_v9/collision/base_link.STL" />
+      <inertia ixx="42.2528214496965" ixy="2.90433873714437E-05" ixz="5.298622447798" iyy="45.7349589120892" iyz="-7.53976926582118E-07" izz="73.6336356175808" />
+    </inertial>
+    <visual>
+      <origin xyz="0 0 0" rpy="0 0 0" />
+      <geometry>
+        <mesh filename="package://alfa_robot_description/meshes/current_robot/visual/base_link.STL" />
+      </geometry>
+      <material name="">
+        <color rgba="0.752941176470588 0.752941176470588 0.752941176470588 1" />
+      </material>
+    </visual>
+    <collision>
+      <origin xyz="0 0 0" rpy="0 0 0" />
+      <geometry>
+        <mesh filename="package://alfa_robot_description/meshes/current_robot/collision/base_link.STL" />
       </geometry>
     </collision>
@@ -41,21 +41,21 @@
   <link name="pitch">
     <inertial>
-      <origin xyz="-0.197223755735604 0.0545002751304143 0.0848583683408157" rpy="0 0 0" />
+      <origin xyz="-0.197223755735604 0.0545002751304142 0.0848583683408171" rpy="0 0 0" />
       <mass value="31.6766900042973" />
-      <inertia ixx="0.518885879634885" ixy="2.02803902279695E-08" ixz="-0.00591642486892729" iyy="0.580169083875299" iyz="3.22538967431134E-07" izz="1.06295541093974" />
-    </inertial>
-    <visual>
-      <origin xyz="0 0 0" rpy="0 0 0" />
-      <geometry>
-        <mesh filename="package://alfa_robot_description/meshes/alfa_robot_v2_arm_v9/visual/pitch.STL" />
-      </geometry>
-      <material name="">
-        <color rgba="0.752941176470588 0.752941176470588 0.752941176470588 1" />
-      </material>
-    </visual>
-    <collision>
-      <origin xyz="0 0 0" rpy="0 0 0" />
-      <geometry>
-        <mesh filename="package://alfa_robot_description/meshes/alfa_robot_v2_arm_v9/collision/pitch.STL" />
+      <inertia ixx="0.518885879634885" ixy="2.02803902282039E-08" ixz="-0.0059164248689273" iyy="0.580169083875299" iyz="3.22538967435459E-07" izz="1.06295541093974" />
+    </inertial>
+    <visual>
+      <origin xyz="0 0 0" rpy="0 0 0" />
+      <geometry>
+        <mesh filename="package://alfa_robot_description/meshes/current_robot/visual/pitch.STL" />
+      </geometry>
+      <material name="">
+        <color rgba="0.752941176470588 0.752941176470588 0.752941176470588 1" />
+      </material>
+    </visual>
+    <collision>
+      <origin xyz="0 0 0" rpy="0 0 0" />
+      <geometry>
+        <mesh filename="package://alfa_robot_description/meshes/current_robot/collision/pitch.STL" />
       </geometry>
     </collision>
@@ -63,21 +63,21 @@
   <link name="turn">
     <inertial>
-      <origin xyz="-0.00958110945289126 -7.73859721442394E-06 1.06018839944043" rpy="0 0 0" />
+      <origin xyz="-0.0095811094528917 -7.73859721447945E-06 1.06018839944043" rpy="0 0 0" />
       <mass value="53.4681885650186" />
-      <inertia ixx="7.9404350019494" ixy="5.99860879545119E-06" ixz="0.185339515626497" iyy="8.17240800709107" iyz="-8.94803411816649E-06" izz="0.75519185821394" />
-    </inertial>
-    <visual>
-      <origin xyz="0 0 0" rpy="0 0 0" />
-      <geometry>
-        <mesh filename="package://alfa_robot_description/meshes/alfa_robot_v2_arm_v9/visual/turn.STL" />
-      </geometry>
-      <material name="">
-        <color rgba="0.752941176470588 0.752941176470588 0.752941176470588 1" />
-      </material>
-    </visual>
-    <collision>
-      <origin xyz="0 0 0" rpy="0 0 0" />
-      <geometry>
-        <mesh filename="package://alfa_robot_description/meshes/alfa_robot_v2_arm_v9/collision/turn.STL" />
+      <inertia ixx="7.9404350019494" ixy="5.99860879539091E-06" ixz="0.185339515626497" iyy="8.17240800709107" iyz="-8.94803411825732E-06" izz="0.75519185821394" />
+    </inertial>
+    <visual>
+      <origin xyz="0 0 0" rpy="0 0 0" />
+      <geometry>
+        <mesh filename="package://alfa_robot_description/meshes/current_robot/visual/turn.STL" />
+      </geometry>
+      <material name="">
+        <color rgba="0.752941176470588 0.752941176470588 0.752941176470588 1" />
+      </material>
+    </visual>
+    <collision>
+      <origin xyz="0 0 0" rpy="0 0 0" />
+      <geometry>
+        <mesh filename="package://alfa_robot_description/meshes/current_robot/collision/turn.STL" />
       </geometry>
     </collision>
@@ -85,26 +85,26 @@
   <link name="updown">
     <inertial>
-      <origin xyz="0.0637333774739139 -2.9260470713055E-09 0.104211014753683" rpy="0 0 0" />
+      <origin xyz="0.0637333774739139 -2.92604740437241E-09 0.104211014753682" rpy="0 0 0" />
       <mass value="24.4167257440598" />
-      <inertia ixx="1.07967195604977" ixy="-1.55435028024514E-08" ixz="-0.00582099906204064" iyy="0.231957862842844" iyz="9.04966240965367E-11" izz="1.26737556353379" />
-    </inertial>
-    <visual>
-      <origin xyz="0 0 0" rpy="0 0 0" />
-      <geometry>
-        <mesh filename="package://alfa_robot_description/meshes/alfa_robot_v2_arm_v9/visual/updown.STL" />
-      </geometry>
-      <material name="">
-        <color rgba="0.752941176470588 0.752941176470588 0.752941176470588 1" />
-      </material>
-    </visual>
-    <collision>
-      <origin xyz="0 0 0" rpy="0 0 0" />
-      <geometry>
-        <mesh filename="package://alfa_robot_description/meshes/alfa_robot_v2_arm_v9/collision/updown.STL" />
-      </geometry>
-    </collision>
-  </link>
-  <!-- ========== LEFT ARM v9 mapped to left_v5_* project names ========== -->
-  <link name="left_v5_link0">
+      <inertia ixx="1.07967195604977" ixy="-1.55435028640832E-08" ixz="-0.00582099906204058" iyy="0.231957862842844" iyz="9.04966113481007E-11" izz="1.26737556353379" />
+    </inertial>
+    <visual>
+      <origin xyz="0 0 0" rpy="0 0 0" />
+      <geometry>
+        <mesh filename="package://alfa_robot_description/meshes/current_robot/visual/updown.STL" />
+      </geometry>
+      <material name="">
+        <color rgba="0.752941176470588 0.752941176470588 0.752941176470588 1" />
+      </material>
+    </visual>
+    <collision>
+      <origin xyz="0 0 0" rpy="0 0 0" />
+      <geometry>
+        <mesh filename="package://alfa_robot_description/meshes/current_robot/collision/updown.STL" />
+      </geometry>
+    </collision>
+  </link>
+  <!-- ========== LEFT ARM mapped to project names ========== -->
+  <link name="left_arm_base">
     <inertial>
       <origin xyz="0 0 0" rpy="0 0 0"/>
@@ -113,185 +113,185 @@
     </inertial>
   </link>
-  <joint name="left_v5_mount" type="fixed">
+  <joint name="left_arm_mount" type="fixed">
     <parent link="updown"/>
-    <child link="left_v5_link0"/>
+    <child link="left_arm_base"/>
     <origin xyz="0.095 0.26 0.2" rpy="0 0 0"/>
   </joint>
-  <link name="left_v5_link1">
-    <inertial>
-      <origin xyz="1.9813263254731E-05 0.00247298217574687 0.0580356323599454" rpy="0 0 0" />
-      <mass value="2.53849365971103" />
-      <inertia ixx="0.00565316591359282" ixy="1.39299660407887E-06" ixz="-2.78630772083778E-06" iyy="0.00554455173094211" iyz="-7.0690628326149E-05" izz="0.00447417412424851" />
-    </inertial>
-    <visual>
-      <origin xyz="0 0 0" rpy="0 0 0" />
-      <geometry>
-        <mesh filename="package://alfa_robot_description/meshes/alfa_robot_v2_arm_v9/visual/leftjoint1.STL" />
-      </geometry>
-      <material name="">
-        <color rgba="0.752941176470588 0.752941176470588 0.752941176470588 1" />
-      </material>
-    </visual>
-    <collision>
-      <origin xyz="0 0 0" rpy="0 0 0" />
-      <geometry>
-        <mesh filename="package://alfa_robot_description/meshes/alfa_robot_v2_arm_v9/collision/leftjoint1.STL" />
-      </geometry>
-    </collision>
-  </link>
-  <joint name="left_v5_joint1" type="revolute">
+  <link name="leftjoint1">
+    <inertial>
+      <origin xyz="1.98132632578396E-05 0.0024729821757461 0.0580356323599247" rpy="0 0 0" />
+      <mass value="2.53849365971092" />
+      <inertia ixx="0.00565316591359222" ixy="1.39299660382164E-06" ixz="-2.78630772107311E-06" iyy="0.00554455173094155" iyz="-7.06906283259906E-05" izz="0.00447417412424819" />
+    </inertial>
+    <visual>
+      <origin xyz="0 0 0" rpy="0 0 0" />
+      <geometry>
+        <mesh filename="package://alfa_robot_description/meshes/current_robot/visual/leftjoint1.STL" />
+      </geometry>
+      <material name="">
+        <color rgba="0.752941176470588 0.752941176470588 0.752941176470588 1" />
+      </material>
+    </visual>
+    <collision>
+      <origin xyz="0 0 0" rpy="0 0 0" />
+      <geometry>
+        <mesh filename="package://alfa_robot_description/meshes/current_robot/collision/leftjoint1.STL" />
+      </geometry>
+    </collision>
+  </link>
+  <joint name="leftjoint1" type="revolute">
     <origin xyz="0 0 0" rpy="0 0 0" />
-    <parent link="left_v5_link0" />
-    <child link="left_v5_link1" />
+    <parent link="left_arm_base" />
+    <child link="leftjoint1" />
     <axis xyz="0 0 1" />
     <limit lower="-2.35619449" upper="2.35619449" effort="120" velocity="1.2" />
   </joint>
-  <link name="left_v5_link2">
-    <inertial>
-      <origin xyz="-3.91993193460394E-09 -0.198242241905549 0.0685963634370443" rpy="0 0 0" />
+  <link name="leftjoint2">
+    <inertial>
+      <origin xyz="-3.91993260073775E-09 -0.198242241905537 0.0685963634370466" rpy="0 0 0" />
       <mass value="13.5734229269593" />
-      <inertia ixx="0.347009291103137" ixy="1.79330552144141E-12" ixz="2.19848829810308E-12" iyy="0.0505989087942829" iyz="4.33554113881788E-12" izz="0.367314390536816" />
-    </inertial>
-    <visual>
-      <origin xyz="0 0 0" rpy="0 0 0" />
-      <geometry>
-        <mesh filename="package://alfa_robot_description/meshes/alfa_robot_v2_arm_v9/visual/leftjoint2.STL" />
-      </geometry>
-      <material name="">
-        <color rgba="0.752941176470588 0.752941176470588 0.752941176470588 1" />
-      </material>
-    </visual>
-    <collision>
-      <origin xyz="0 0 0" rpy="0 0 0" />
-      <geometry>
-        <mesh filename="package://alfa_robot_description/meshes/alfa_robot_v2_arm_v9/collision/leftjoint2.STL" />
-      </geometry>
-    </collision>
-  </link>
-  <joint name="left_v5_joint2" type="revolute">
-    <origin xyz="0 0.0825 0.0579999999999996" rpy="-1.5707963267949 0 0" />
-    <parent link="left_v5_link1" />
-    <child link="left_v5_link2" />
+      <inertia ixx="0.347009291103137" ixy="1.79329294469621E-12" ixz="2.19848376530362E-12" iyy="0.0505989087942828" iyz="4.33552705015945E-12" izz="0.367314390536816" />
+    </inertial>
+    <visual>
+      <origin xyz="0 0 0" rpy="0 0 0" />
+      <geometry>
+        <mesh filename="package://alfa_robot_description/meshes/current_robot/visual/leftjoint2.STL" />
+      </geometry>
+      <material name="">
+        <color rgba="0.752941176470588 0.752941176470588 0.752941176470588 1" />
+      </material>
+    </visual>
+    <collision>
+      <origin xyz="0 0 0" rpy="0 0 0" />
+      <geometry>
+        <mesh filename="package://alfa_robot_description/meshes/current_robot/collision/leftjoint2.STL" />
+      </geometry>
+    </collision>
+  </link>
+  <joint name="leftjoint2" type="revolute">
+    <origin xyz="0 0.0825 0.058" rpy="-1.5708 0 0" />
+    <parent link="leftjoint1" />
+    <child link="leftjoint2" />
     <axis xyz="0 0 1" />
     <limit lower="-3.14159265" upper="3.14159265" effort="120" velocity="1.2" />
   </joint>
-  <link name="left_v5_link3">
-    <inertial>
-      <origin xyz="4.24816812838458E-08 -0.171995906773402 -0.0220559637033981" rpy="0 0 0" />
-      <mass value="5.37152510221438" />
-      <inertia ixx="0.103379389320522" ixy="1.01375731816284E-08" ixz="4.8440173396198E-09" iyy="0.0137404008500263" iyz="0.000240093301068499" izz="0.114911955120257" />
-    </inertial>
-    <visual>
-      <origin xyz="0 0 0" rpy="0 0 0" />
-      <geometry>
-        <mesh filename="package://alfa_robot_description/meshes/alfa_robot_v2_arm_v9/visual/leftjoint3.STL" />
-      </geometry>
-      <material name="">
-        <color rgba="0.752941176470588 0.752941176470588 0.752941176470588 1" />
-      </material>
-    </visual>
-    <collision>
-      <origin xyz="0 0 0" rpy="0 0 0" />
-      <geometry>
-        <mesh filename="package://alfa_robot_description/meshes/alfa_robot_v2_arm_v9/collision/leftjoint3.STL" />
-      </geometry>
-    </collision>
-  </link>
-  <joint name="left_v5_joint3" type="revolute">
+  <link name="leftjoint3">
+    <inertial>
+      <origin xyz="2.86018788653308E-08 -0.174995964436896 -0.0214654505916678" rpy="0 0 0" />
+      <mass value="5.46918956371602" />
+      <inertia ixx="0.102635037762556" ixy="1.82331494669218E-08" ixz="3.03709958770067E-09" iyy="0.0138225294833702" iyz="4.39575520960004E-05" izz="0.114289616262011" />
+    </inertial>
+    <visual>
+      <origin xyz="0 0 0" rpy="0 0 0" />
+      <geometry>
+        <mesh filename="package://alfa_robot_description/meshes/current_robot/visual/leftjoint3.STL" />
+      </geometry>
+      <material name="">
+        <color rgba="0.752941176470588 0.752941176470588 0.752941176470588 1" />
+      </material>
+    </visual>
+    <collision>
+      <origin xyz="0 0 0" rpy="0 0 0" />
+      <geometry>
+        <mesh filename="package://alfa_robot_description/meshes/current_robot/collision/leftjoint3.STL" />
+      </geometry>
+    </collision>
+  </link>
+  <joint name="leftjoint3" type="revolute">
     <origin xyz="0 -0.4 0.008" rpy="0 0 0" />
-    <parent link="left_v5_link2" />
-    <child link="left_v5_link3" />
+    <parent link="leftjoint2" />
+    <child link="leftjoint3" />
     <axis xyz="0 0 1" />
     <limit lower="-3.14159265" upper="3.14159265" effort="100" velocity="1.2" />
   </joint>
-  <link name="left_v5_link4">
-    <inertial>
-      <origin xyz="1.86328980931183E-05 0.00232765205467672 0.0541835839509776" rpy="0 0 0" />
-      <mass value="2.69701889029267" />
-      <inertia ixx="0.00655846785174234" ixy="1.39368136512847E-06" ixz="-2.78625493222266E-06" iyy="0.00644984634538746" iyz="-7.06885588830852E-05" izz="0.00474081047943518" />
-    </inertial>
-    <visual>
-      <origin xyz="0 0 0" rpy="0 0 0" />
-      <geometry>
-        <mesh filename="package://alfa_robot_description/meshes/alfa_robot_v2_arm_v9/visual/leftjoint4.STL" />
-      </geometry>
-      <material name="">
-        <color rgba="0.752941176470588 0.752941176470588 0.752941176470588 1" />
-      </material>
-    </visual>
-    <collision>
-      <origin xyz="0 0 0" rpy="0 0 0" />
-      <geometry>
-        <mesh filename="package://alfa_robot_description/meshes/alfa_robot_v2_arm_v9/collision/leftjoint4.STL" />
-      </geometry>
-    </collision>
-  </link>
-  <joint name="left_v5_joint4" type="revolute">
-    <origin xyz="0 -0.34 0.021" rpy="0 0 3.14159265" />
-    <parent link="left_v5_link3" />
-    <child link="left_v5_link4" />
+  <link name="leftjoint4">
+    <inertial>
+      <origin xyz="1.79301766545237E-05 0.0022398818670486 0.0513862987308302" rpy="0 0 0" />
+      <mass value="2.80270206383319" />
+      <inertia ixx="0.00725799360950605" ixy="1.39369533421895E-06" ixz="-2.78625386086696E-06" iyy="0.00714937209205323" iyz="-7.06885588698108E-05" izz="0.00491856957816283" />
+    </inertial>
+    <visual>
+      <origin xyz="0 0 0" rpy="0 0 0" />
+      <geometry>
+        <mesh filename="package://alfa_robot_description/meshes/current_robot/visual/leftjoint4.STL" />
+      </geometry>
+      <material name="">
+        <color rgba="0.752941176470588 0.752941176470588 0.752941176470588 1" />
+      </material>
+    </visual>
+    <collision>
+      <origin xyz="0 0 0" rpy="0 0 0" />
+      <geometry>
+        <mesh filename="package://alfa_robot_description/meshes/current_robot/collision/leftjoint4.STL" />
+      </geometry>
+    </collision>
+  </link>
+  <joint name="leftjoint4" type="revolute">
+    <origin xyz="0 -0.34 0.036" rpy="0 0 3.14159265" />
+    <parent link="leftjoint3" />
+    <child link="leftjoint4" />
     <axis xyz="0 0 1" />
     <limit lower="-3.14159265" upper="3.14159265" effort="60" velocity="1.5" />
   </joint>
-  <link name="left_v5_link5">
-    <inertial>
-      <origin xyz="0.00232761885815602 1.86282477868636E-05 -0.0541835932362763" rpy="0 0 0" />
-      <mass value="2.69701788961671" />
-      <inertia ixx="0.00644984661938229" ixy="1.39391456321868E-06" ixz="7.06885192212674E-05" iyy="0.00655846677978978" iyz="2.78593765675197E-06" izz="0.00474081002137946" />
-    </inertial>
-    <visual>
-      <origin xyz="0 0 0" rpy="0 0 0" />
-      <geometry>
-        <mesh filename="package://alfa_robot_description/meshes/alfa_robot_v2_arm_v9/visual/leftjoint5.STL" />
-      </geometry>
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