Commit message: refactor(robot): 收口新机械臂命名与仓库资产
- 将当前机械臂模型收口到 current_robot mesh 和无版本语义的关节、group、controller 命名。
- 同步 description、MoveIt、bringup、execution bridge、scene service、MuJoCo 与 benchmark 脚本中的新命名。
- 移除旧代际 mesh、废弃 URDF 入口、pick_ik/trac_ik 依赖包和旧 IK 安装脚本。
- 更新 IK 服务口径、命名护栏文档和协作日志，保留当前 BioIK/KDL 主线能力。

验证：
- git diff --cached --check 通过。
- colcon build --packages-select alfa_robot_description robot_motion_scene_service alfa_robot_moveit_config alfa_robot_bringup alfa_robot_execution_bridge alfa_robot_benchmarks --symlink-install --cmake-args -DBUILD_TESTING=OFF 通过。
- colcon build --packages-select robot_motion_scene_service alfa_robot_moveit_config --symlink-install --cmake-args -DBUILD_TESTING=ON 通过。
- colcon test --packages-select robot_motion_scene_service alfa_robot_moveit_config --return-code-on-test-failure 通过；colcon test-result --verbose 显示 15 tests, 0 errors, 0 failures。

Co-Authored-By: Codex <codex@openai.com>

File: ros2_ws/src/alfa_robot_description/urdf/alfa_robot/alfa_robot_macro.ros2_control.xacro (robot description, xacro)
@@ -15,16 +15,16 @@
                turn_initial:=0.0
                updown_initial:=0.0
-               left_v5_joint1_initial:=0.0
-               left_v5_joint2_initial:=0.0
-               left_v5_joint3_initial:=0.0
-               left_v5_joint4_initial:=0.0
-               left_v5_joint5_initial:=0.0
-               left_v5_joint6_initial:=0.0
-               right_v5_joint1_initial:=0.0
-               right_v5_joint2_initial:=0.0
-               right_v5_joint3_initial:=0.0
-               right_v5_joint4_initial:=0.0
-               right_v5_joint5_initial:=0.0
-               right_v5_joint6_initial:=0.0"
+               leftjoint1_initial:=0.0
+               leftjoint2_initial:=0.0
+               leftjoint3_initial:=0.0
+               leftjoint4_initial:=0.0
+               leftjoint5_initial:=0.0
+               leftjoint6_initial:=0.0
+               rightjoint1_initial:=0.0
+               rightjoint2_initial:=0.0
+               rightjoint3_initial:=0.0
+               rightjoint4_initial:=0.0
+               rightjoint5_initial:=0.0
+               rightjoint6_initial:=0.0"
                >
     <ros2_control name="${name}" type="system">
@@ -89,6 +89,6 @@
         <state_interface name="acceleration"/>
       </joint>
-      <!-- v5 proxy arms (position controlled) -->
-      <xacro:macro name="v5_proxy_control_joint" params="joint_name lower upper velocity initial_value:=0.0">
+      <!-- dual arms (position controlled) -->
+      <xacro:macro name="arm_control_joint" params="joint_name lower upper velocity initial_value:=0.0">
         <joint name="${prefix}${joint_name}">
           <command_interface name="position">
@@ -103,16 +103,16 @@
         </joint>
       </xacro:macro>
-      <xacro:v5_proxy_control_joint joint_name="left_v5_joint1" lower="-0.0" upper="0.0" velocity="1.2" initial_value="${left_v5_joint1_initial}"/>
-      <xacro:v5_proxy_control_joint joint_name="left_v5_joint2" lower="-3.14159265" upper="3.14159265" velocity="1.2" initial_value="${left_v5_joint2_initial}"/>
-      <xacro:v5_proxy_control_joint joint_name="left_v5_joint3" lower="-3.14159265" upper="3.14159265" velocity="1.2" initial_value="${left_v5_joint3_initial}"/>
-      <xacro:v5_proxy_control_joint joint_name="left_v5_joint4" lower="-3.14159265" upper="3.14159265" velocity="1.5" initial_value="${left_v5_joint4_initial}"/>
-      <xacro:v5_proxy_control_joint joint_name="left_v5_joint5" lower="-3.14159265" upper="3.14159265" velocity="1.5" initial_value="${left_v5_joint5_initial}"/>
-      <xacro:v5_proxy_control_joint joint_name="left_v5_joint6" lower="-3.14159265" upper="3.14159265" velocity="1.5" initial_value="${left_v5_joint6_initial}"/>
-      <xacro:v5_proxy_control_joint joint_name="right_v5_joint1" lower="-0.0" upper="0.0" velocity="1.2" initial_value="${right_v5_joint1_initial}"/>
-      <xacro:v5_proxy_control_joint joint_name="right_v5_joint2" lower="-3.14159265" upper="3.14159265" velocity="1.2" initial_value="${right_v5_joint2_initial}"/>
-      <xacro:v5_proxy_control_joint joint_name="right_v5_joint3" lower="-3.14159265" upper="3.14159265" velocity="1.2" initial_value="${right_v5_joint3_initial}"/>
-      <xacro:v5_proxy_control_joint joint_name="right_v5_joint4" lower="-3.14159265" upper="3.14159265" velocity="1.5" initial_value="${right_v5_joint4_initial}"/>
-      <xacro:v5_proxy_control_joint joint_name="right_v5_joint5" lower="-3.14159265" upper="3.14159265" velocity="1.5" initial_value="${right_v5_joint5_initial}"/>
-      <xacro:v5_proxy_control_joint joint_name="right_v5_joint6" lower="-3.14159265" upper="3.14159265" velocity="1.5" initial_value="${right_v5_joint6_initial}"/>
+      <xacro:arm_control_joint joint_name="leftjoint1" lower="-0.0" upper="0.0" velocity="1.2" initial_value="${leftjoint1_initial}"/>
+      <xacro:arm_control_joint joint_name="leftjoint2" lower="-3.14159265" upper="3.14159265" velocity="1.2" initial_value="${leftjoint2_initial}"/>
+      <xacro:arm_control_joint joint_name="leftjoint3" lower="-3.14159265" upper="3.14159265" velocity="1.2" initial_value="${leftjoint3_initial}"/>
+      <xacro:arm_control_joint joint_name="leftjoint4" lower="-3.14159265" upper="3.14159265" velocity="1.5" initial_value="${leftjoint4_initial}"/>
+      <xacro:arm_control_joint joint_name="leftjoint5" lower="-3.14159265" upper="3.14159265" velocity="1.5" initial_value="${leftjoint5_initial}"/>
+      <xacro:arm_control_joint joint_name="leftjoint6" lower="-3.14159265" upper="3.14159265" velocity="1.5" initial_value="${leftjoint6_initial}"/>
+      <xacro:arm_control_joint joint_name="rightjoint1" lower="-0.0" upper="0.0" velocity="1.2" initial_value="${rightjoint1_initial}"/>
+      <xacro:arm_control_joint joint_name="rightjoint2" lower="-3.14159265" upper="3.14159265" velocity="1.2" initial_value="${rightjoint2_initial}"/>
+      <xacro:arm_control_joint joint_name="rightjoint3" lower="-3.14159265" upper="3.14159265" velocity="1.2" initial_value="${rightjoint3_initial}"/>
+      <xacro:arm_control_joint joint_name="rightjoint4" lower="-3.14159265" upper="3.14159265" velocity="1.5" initial_value="${rightjoint4_initial}"/>
+      <xacro:arm_control_joint joint_name="rightjoint5" lower="-3.14159265" upper="3.14159265" velocity="1.5" initial_value="${rightjoint5_initial}"/>
+      <xacro:arm_control_joint joint_name="rightjoint6" lower="-3.14159265" upper="3.14159265" velocity="1.5" initial_value="${rightjoint6_initial}"/>
     </ros2_control>
     <xacro:if value="$(arg sim_gazebo_classic)">
