Commit message: fix(v3): 对齐V3.1.1 Demo模型合同 Refs MOTION-94

File: ros2_ws/src/alfa_robot_description/urdf/alfa_robot.urdf.xacro (robot description, xacro)
@@ -5,17 +5,20 @@
   <xacro:arg name="mock_sensor_commands" default="true"/>
   <xacro:arg name="arm_mount_forward_offset" default="0"/>
-  <xacro:arg name="updown_initial" default="0.0"/>
+  <xacro:arg name="base_link_x" default="0.195"/>
+  <xacro:arg name="base_link_y" default="0.015"/>
+  <xacro:arg name="base_link_z" default="0.400"/>
+  <xacro:arg name="updown_initial" default="-0.5"/>
   <xacro:arg name="head_joint_initial" default="0.0"/>
-  <xacro:arg name="left_joint1_initial" default="-1.57079632679"/>
-  <xacro:arg name="left_joint2_initial" default="-1.57079632679"/>
-  <xacro:arg name="left_joint3_initial" default="0.0"/>
-  <xacro:arg name="left_joint4_initial" default="-1.57079632679"/>
+  <xacro:arg name="left_joint1_initial" default="2.61799387799"/>
+  <xacro:arg name="left_joint2_initial" default="1.57079632679"/>
+  <xacro:arg name="left_joint3_initial" default="-0.0872664625997"/>
+  <xacro:arg name="left_joint4_initial" default="2.09439510239"/>
   <xacro:arg name="left_joint5_initial" default="0.0"/>
   <xacro:arg name="left_joint6_initial" default="0.0"/>
   <xacro:arg name="left_joint7_initial" default="0.0"/>
-  <xacro:arg name="right_joint1_initial" default="-1.57079632679"/>
+  <xacro:arg name="right_joint1_initial" default="-2.61799387799"/>
   <xacro:arg name="right_joint2_initial" default="-1.57079632679"/>
-  <xacro:arg name="right_joint3_initial" default="0.0"/>
-  <xacro:arg name="right_joint4_initial" default="-1.57079632679"/>
+  <xacro:arg name="right_joint3_initial" default="0.0872664625997"/>
+  <xacro:arg name="right_joint4_initial" default="-2.09439510239"/>
   <xacro:arg name="right_joint5_initial" default="0.0"/>
   <xacro:arg name="right_joint6_initial" default="0.0"/>
@@ -23,10 +26,10 @@
   <xacro:include filename="$(find alfa_robot_description)/urdf/alfa_robot/alfa_robot_macro.ros2_control.xacro"/>
   <xacro:property name="arm_mount_forward_offset_value" value="$(arg arm_mount_forward_offset)"/>
-  <xacro:include filename="$(find alfa_robot_description)/urdf/alfa_robot/robot_v3_0_9.xacro"/>
-  <link name="world"/>
-  <joint name="world_to_base" type="fixed">
-    <parent link="world"/>
+  <xacro:include filename="$(find alfa_robot_description)/urdf/alfa_robot/robot_v3_1_1.xacro"/>
+  <link name="base_footprint"/>
+  <joint name="base_footprint_to_base_link" type="fixed">
+    <parent link="base_footprint"/>
     <child link="base_link"/>
-    <origin xyz="0 0 0" rpy="0 0 0"/>
+    <origin xyz="$(arg base_link_x) $(arg base_link_y) $(arg base_link_z)" rpy="0 0 0"/>
   </joint>
   <link name="base_link"/>
@@ -35,5 +38,5 @@
     <child link="model_base"/>
     <origin
-      xyz="${-0.190000017371 + float(arm_mount_forward_offset_value)} 6.50500004219e-09 0.648299964909"
+      xyz="${-0.174000020720362 + float(arm_mount_forward_offset_value)} 6.50500007062811e-09 0.802299964909"
       rpy="1.5707963 0 1.57079632679"/>
   </joint>

File: ros2_ws/src/alfa_robot_description/urdf/alfa_robot/alfa_robot_macro.ros2_control.xacro (robot description, xacro)
@@ -6,17 +6,17 @@
                use_mock_hardware:=true
                mock_sensor_commands:=true
-               updown_initial:=0.0
+               updown_initial:=-0.5
                head_joint_initial:=0.0
-               left_joint1_initial:=-1.57079632679
-               left_joint2_initial:=-1.57079632679
-               left_joint3_initial:=0.0
-               left_joint4_initial:=-1.57079632679
+               left_joint1_initial:=2.61799387799
+               left_joint2_initial:=1.57079632679
+               left_joint3_initial:=-0.0872664625997
+               left_joint4_initial:=2.09439510239
                left_joint5_initial:=0.0
                left_joint6_initial:=0.0
                left_joint7_initial:=0.0
-               right_joint1_initial:=-1.57079632679
+               right_joint1_initial:=-2.61799387799
                right_joint2_initial:=-1.57079632679
-               right_joint3_initial:=0.0
-               right_joint4_initial:=-1.57079632679
+               right_joint3_initial:=0.0872664625997
+               right_joint4_initial:=-2.09439510239
                right_joint5_initial:=0.0
                right_joint6_initial:=0.0
@@ -27,5 +27,5 @@
         <param name="mock_sensor_commands">${mock_sensor_commands}</param>
       </hardware>
-      <xacro:macro name="arm_control_joint" params="joint_name initial_value lower upper">
+      <xacro:macro name="control_joint" params="joint_name initial_value lower upper">
         <joint name="${prefix}${joint_name}">
           <command_interface name="position">
@@ -39,20 +39,31 @@
         </joint>
       </xacro:macro>
-      <xacro:arm_control_joint joint_name="updown" initial_value="${updown_initial}" lower="-1.0" upper="0.0"/>
-      <xacro:arm_control_joint joint_name="head_joint" initial_value="${head_joint_initial}" lower="-1.57" upper="1.57"/>
-      <xacro:arm_control_joint joint_name="left_joint1" initial_value="${left_joint1_initial}" lower="-3.14159265" upper="3.14159265"/>
-      <xacro:arm_control_joint joint_name="left_joint2" initial_value="${left_joint2_initial}" lower="-1.83259571" upper="1.83259571"/>
-      <xacro:arm_control_joint joint_name="left_joint3" initial_value="${left_joint3_initial}" lower="-3.14159265" upper="3.14159265"/>
-      <xacro:arm_control_joint joint_name="left_joint4" initial_value="${left_joint4_initial}" lower="-2.53072742" upper="2.53072742"/>
-      <xacro:arm_control_joint joint_name="left_joint5" initial_value="${left_joint5_initial}" lower="-3.14159265" upper="3.14159265"/>
-      <xacro:arm_control_joint joint_name="left_joint6" initial_value="${left_joint6_initial}" lower="-1.91986218" upper="1.91986218"/>
-      <xacro:arm_control_joint joint_name="left_joint7" initial_value="${left_joint7_initial}" lower="-3.14159265" upper="3.14159265"/>
-      <xacro:arm_control_joint joint_name="right_joint1" initial_value="${right_joint1_initial}" lower="-3.14159265" upper="3.14159265"/>
-      <xacro:arm_control_joint joint_name="right_joint2" initial_value="${right_joint2_initial}" lower="-1.83259571" upper="1.83259571"/>
-      <xacro:arm_control_joint joint_name="right_joint3" initial_value="${right_joint3_initial}" lower="-3.14159265" upper="3.14159265"/>
-      <xacro:arm_control_joint joint_name="right_joint4" initial_value="${right_joint4_initial}" lower="-2.53072742" upper="2.53072742"/>
-      <xacro:arm_control_joint joint_name="right_joint5" initial_value="${right_joint5_initial}" lower="-3.14159265" upper="3.14159265"/>
-      <xacro:arm_control_joint joint_name="right_joint6" initial_value="${right_joint6_initial}" lower="-1.91986218" upper="1.91986218"/>
-      <xacro:arm_control_joint joint_name="right_joint7" initial_value="${right_joint7_initial}" lower="-3.14159265" upper="3.14159265"/>
+      <xacro:control_joint joint_name="rear_suspension_joint" initial_value="0.085" lower="0" upper="0.17"/>
+      <xacro:control_joint joint_name="front_left_steering_joint" initial_value="0" lower="-1.57" upper="1.57"/>
+      <xacro:control_joint joint_name="front_left_wheel_joint" initial_value="0" lower="-1.57" upper="1.57"/>
+      <xacro:control_joint joint_name="front_right_steering_joint" initial_value="0" lower="-1.57" upper="1.57"/>
+      <xacro:control_joint joint_name="front_right_wheel_joint" initial_value="0" lower="-1.57" upper="1.57"/>
+      <xacro:control_joint joint_name="rear_left_steering_joint" initial_value="0" lower="-1.57" upper="1.57"/>
+      <xacro:control_joint joint_name="rear_left_wheel_joint" initial_value="0" lower="-1.57" upper="1.57"/>
+      <xacro:control_joint joint_name="rear_right_steering_joint" initial_value="0" lower="-1.57" upper="1.57"/>
+      <xacro:control_joint joint_name="rear_right_wheel_joint" initial_value="0" lower="-1.57" upper="1.57"/>
+      <xacro:control_joint joint_name="updown" initial_value="${updown_initial}" lower="-1" upper="0"/>
+      <xacro:control_joint joint_name="head_joint" initial_value="${head_joint_initial}" lower="-1.57" upper="1.57"/>
+      <xacro:control_joint joint_name="left_joint1" initial_value="${left_joint1_initial}" lower="-3.14159265" upper="3.14159265"/>
+      <xacro:control_joint joint_name="left_joint2" initial_value="${left_joint2_initial}" lower="-1.8325957145940461" upper="1.8325957145940461"/>
+      <xacro:control_joint joint_name="left_joint3" initial_value="${left_joint3_initial}" lower="-3.14159265" upper="3.14159265"/>
+      <xacro:control_joint joint_name="left_joint4" initial_value="${left_joint4_initial}" lower="-2.53072742" upper="2.53072742"/>
+      <xacro:control_joint joint_name="left_joint5" initial_value="${left_joint5_initial}" lower="-3.14159265" upper="3.14159265"/>
+      <xacro:control_joint joint_name="left_joint6" initial_value="${left_joint6_initial}" lower="-1.91986218" upper="1.91986218"/>
+      <xacro:control_joint joint_name="left_joint7" initial_value="${left_joint7_initial}" lower="-3.14159265" upper="3.14159265"/>
+      <xacro:control_joint joint_name="left_hand_joint" initial_value="0" lower="0" upper="0.1"/>
+      <xacro:control_joint joint_name="right_joint1" initial_value="${right_joint1_initial}" lower="-3.14159265" upper="3.14159265"/>
+      <xacro:control_joint joint_name="right_joint2" initial_value="${right_joint2_initial}" lower="-1.8325957145940461" upper="1.8325957145940461"/>
+      <xacro:control_joint joint_name="right_joint3" initial_value="${right_joint3_initial}" lower="-3.14159265" upper="3.14159265"/>
+      <xacro:control_joint joint_name="right_joint4" initial_value="${right_joint4_initial}" lower="-2.53072742" upper="2.53072742"/>
+      <xacro:control_joint joint_name="right_joint5" initial_value="${right_joint5_initial}" lower="-3.14159265" upper="3.14159265"/>
+      <xacro:control_joint joint_name="right_joint6" initial_value="${right_joint6_initial}" lower="-1.91986218" upper="1.91986218"/>
+      <xacro:control_joint joint_name="right_joint7" initial_value="${right_joint7_initial}" lower="-3.14159265" upper="3.14159265"/>
+      <xacro:control_joint joint_name="right_hand_joint" initial_value="0" lower="0" upper="0.1"/>
     </ros2_control>
   </xacro:macro>

Commit message: feat(v3): 统一双臂对称零位与装卸姿态 Refs MOTION-204

File: ros2_ws/src/alfa_robot_description/urdf/alfa_robot.urdf.xacro (robot description, xacro)
@@ -18,9 +18,9 @@
   <xacro:arg name="left_joint6_initial" default="-0.69813170079773"/>
   <xacro:arg name="left_joint7_initial" default="0.0"/>
-  <xacro:arg name="right_joint1_initial" default="0.43633231299858"/>
+  <xacro:arg name="right_joint1_initial" default="-2.70526034059121"/>
   <xacro:arg name="right_joint2_initial" default="-1.832595714594046"/>
   <xacro:arg name="right_joint3_initial" default="-0.34906585039887"/>
   <xacro:arg name="right_joint4_initial" default="1.57079632679490"/>
-  <xacro:arg name="right_joint5_initial" default="-1.57079632679490"/>
+  <xacro:arg name="right_joint5_initial" default="1.57079632679490"/>
   <xacro:arg name="right_joint6_initial" default="0.69813170079773"/>
   <xacro:arg name="right_joint7_initial" default="0.0"/>

File: ros2_ws/src/alfa_robot_description/urdf/alfa_robot/alfa_robot_macro.ros2_control.xacro (robot description, xacro)
@@ -17,9 +17,9 @@
                left_joint6_initial:=-0.69813170079773
                left_joint7_initial:=0.0
-               right_joint1_initial:=0.43633231299858
+               right_joint1_initial:=-2.70526034059121
                right_joint2_initial:=-1.832595714594046
                right_joint3_initial:=-0.34906585039887
                right_joint4_initial:=1.57079632679490
-               right_joint5_initial:=-1.57079632679490
+               right_joint5_initial:=1.57079632679490
                right_joint6_initial:=0.69813170079773
                right_joint7_initial:=0.0

File: ros2_ws/src/alfa_robot_description/urdf/alfa_robot/robot_v3_1_1.xacro (robot description, xacro)
@@ -532,5 +532,5 @@
   </joint>
   <joint name="right_joint1" type="revolute">
-    <origin xyz="-0.33054221 -0.181 1.3500054" rpy="0 -1.3089969 0" />
+    <origin xyz="-0.33054221 -0.181 1.3500054" rpy="0 1.3089969 3.1415927" />
     <parent link="right_arm_base" />
     <child link="right_joint1" />
@@ -560,5 +560,5 @@
   </joint>
   <joint name="right_joint5" type="revolute">
-    <origin xyz="-0.22457775 0.060175428 0.068" rpy="-1.5707963 0 1.3089969" />
+    <origin xyz="-0.22457775 0.060175428 0.068" rpy="1.5707963 0 -1.8325957" />
     <parent link="right_joint4" />
     <child link="right_joint5" />
