Commit message: test(v3): lock live golden 25 of 25 regression

File: ros2_ws/src/alfa_robot_description/urdf/alfa_robot.urdf.xacro (robot description, xacro)
@@ -19,7 +19,7 @@
   <xacro:arg name="left_joint7_initial" default="0.0"/>
   <xacro:arg name="right_joint1_initial" default="-2.70526034059121"/>
-  <xacro:arg name="right_joint2_initial" default="1.832595714594046"/>
+  <xacro:arg name="right_joint2_initial" default="-1.832595714594046"/>
   <xacro:arg name="right_joint3_initial" default="-0.34906585039887"/>
-  <xacro:arg name="right_joint4_initial" default="-1.57079632679490"/>
+  <xacro:arg name="right_joint4_initial" default="1.57079632679490"/>
   <xacro:arg name="right_joint5_initial" default="1.57079632679490"/>
   <xacro:arg name="right_joint6_initial" default="0.69813170079773"/>

File: ros2_ws/src/alfa_robot_description/urdf/alfa_robot/alfa_robot_macro.ros2_control.xacro (robot description, xacro)
@@ -18,7 +18,7 @@
                left_joint7_initial:=0.0
                right_joint1_initial:=-2.70526034059121
-               right_joint2_initial:=1.832595714594046
+               right_joint2_initial:=-1.832595714594046
                right_joint3_initial:=-0.34906585039887
-               right_joint4_initial:=-1.57079632679490
+               right_joint4_initial:=1.57079632679490
                right_joint5_initial:=1.57079632679490
                right_joint6_initial:=0.69813170079773

File: ros2_ws/src/alfa_robot_description/urdf/alfa_robot/robot_v3_1_1.xacro (robot description, xacro)
@@ -294,5 +294,5 @@
     </collision>
   </link>
-  <link name="right_link1">
+  <link name="right_joint1">
     <inertial>
       <origin xyz="0.026713078 -0.00035041598 0.12770383" rpy="0 0 0" />
@@ -313,5 +313,5 @@
     </collision>
   </link>
-  <link name="right_link2">
+  <link name="right_joint2">
     <inertial>
       <origin xyz="-0.16472334 -1.1230144e-08 -0.040000126" rpy="0 0 0" />
@@ -332,5 +332,5 @@
     </collision>
   </link>
-  <link name="right_link3">
+  <link name="right_joint3">
     <inertial>
       <origin xyz="-5.896457e-08 9.5061022e-10 0.23006341" rpy="0 0 0" />
@@ -351,5 +351,5 @@
     </collision>
   </link>
-  <link name="right_link4">
+  <link name="right_joint4">
     <inertial>
       <origin xyz="-0.12628065 0.0338368 0.067995266" rpy="0 0 0" />
@@ -370,5 +370,5 @@
     </collision>
   </link>
-  <link name="right_link5">
+  <link name="right_joint5">
     <inertial>
       <origin xyz="-0.026166805 0 0.12943329" rpy="0 0 0" />
@@ -389,5 +389,5 @@
     </collision>
   </link>
-  <link name="right_link6">
+  <link name="right_joint6">
     <inertial>
       <origin xyz="-0.05437806 0 -0.061500007" rpy="0 0 0" />
@@ -409,5 +409,5 @@
   </link>
   <xacro:call macro="v3_$(arg end_effector)" side="right" />
-  <link name="left_link1">
+  <link name="left_joint1">
     <inertial>
       <origin xyz="0.026713079 -0.00035041871 0.12770383" rpy="0 0 0" />
@@ -428,5 +428,5 @@
     </collision>
   </link>
-  <link name="left_link2">
+  <link name="left_joint2">
     <inertial>
       <origin xyz="0.16472335 1.2730856e-08 -0.040000127" rpy="0 0 0" />
@@ -447,5 +447,5 @@
     </collision>
   </link>
-  <link name="left_link3">
+  <link name="left_joint3">
     <inertial>
       <origin xyz="-5.9080015e-08 2.5764869e-09 0.23006341" rpy="0 0 0" />
@@ -466,5 +466,5 @@
     </collision>
   </link>
-  <link name="left_link4">
+  <link name="left_joint4">
     <inertial>
       <origin xyz="0.12628066 0.033836802 0.068004734" rpy="0 0 0" />
@@ -485,5 +485,5 @@
     </collision>
   </link>
-  <link name="left_link5">
+  <link name="left_joint5">
     <inertial>
       <origin xyz="-0.026166799 2.9314955e-10 0.12943328" rpy="0 0 0" />
@@ -504,5 +504,5 @@
     </collision>
   </link>
-  <link name="left_link6">
+  <link name="left_joint6">
     <inertial>
       <origin xyz="0.054378045 -1.1235669e-09 -0.061499998" rpy="0 0 0" />
@@ -532,100 +532,100 @@
   </joint>
   <joint name="right_joint1" type="revolute">
-    <origin xyz="-0.33054221 -0.181 1.3500054" rpy="0 -1.3089969 0" />
+    <origin xyz="-0.33054221 -0.181 1.3500054" rpy="0 1.3089969 3.1415927" />
     <parent link="right_arm_base" />
-    <child link="right_link1" />
-    <axis xyz="0 0 1" />
-    <limit lower="-3.14159265" upper="3.14159265" effort="647" velocity="1.309" />
+    <child link="right_joint1" />
+    <axis xyz="0 0 1" />
+    <limit lower="-3.14159265" upper="3.14159265" effort="10" velocity="5" />
   </joint>
   <joint name="right_joint2" type="revolute">
     <origin xyz="0.039999999 0 0.1512" rpy="0 1.5707963 0" />
-    <parent link="right_link1" />
-    <child link="right_link2" />
-    <axis xyz="0 0 1" />
-    <limit lower="-1.8325957145940461" upper="1.8325957145940461" effort="647" velocity="1.309" />
+    <parent link="right_joint1" />
+    <child link="right_joint2" />
+    <axis xyz="0 0 1" />
+    <limit lower="-1.8325957145940461" upper="1.8325957145940461" effort="10" velocity="5" />
   </joint>
   <joint name="right_joint3" type="revolute">
     <origin xyz="-0.1795 0 -0.040000001" rpy="0 -1.5707963 0" />
-    <parent link="right_link2" />
-    <child link="right_link3" />
-    <axis xyz="0 0 1" />
-    <limit lower="-3.14159265" upper="3.14159265" effort="484" velocity="1.309" />
+    <parent link="right_joint2" />
+    <child link="right_joint3" />
+    <axis xyz="0 0 1" />
+    <limit lower="-3.14159265" upper="3.14159265" effort="10" velocity="5" />
   </joint>
   <joint name="right_joint4" type="revolute">
     <origin xyz="-1.2287747e-09 0.068 0.3265" rpy="1.5707963 1.3089969 0" />
-    <parent link="right_link3" />
-    <child link="right_link4" />
-    <axis xyz="0 0 1" />
-    <limit lower="-2.53072742" upper="2.53072742" effort="459" velocity="1.749" />
+    <parent link="right_joint3" />
+    <child link="right_joint4" />
+    <axis xyz="0 0 1" />
+    <limit lower="-2.53072742" upper="2.53072742" effort="10" velocity="5" />
   </joint>
   <joint name="right_joint5" type="revolute">
-    <origin xyz="-0.22457775 0.060175428 0.068" rpy="-1.5707963 0 1.3089969" />
-    <parent link="right_link4" />
-    <child link="right_link5" />
-    <axis xyz="0 0 1" />
-    <limit lower="-3.14159265" upper="3.14159265" effort="217" velocity="2.618" />
+    <origin xyz="-0.22457775 0.060175428 0.068" rpy="1.5707963 0 -1.8325957" />
+    <parent link="right_joint4" />
+    <child link="right_joint5" />
+    <axis xyz="0 0 1" />
+    <limit lower="-3.14159265" upper="3.14159265" effort="10" velocity="5" />
   </joint>
   <joint name="right_joint6" type="revolute">
     <origin xyz="0.061499999 0 0.2415" rpy="0 1.5707963 0" />
-    <parent link="right_link5" />
-    <child link="right_link6" />
-    <axis xyz="0 0 1" />
-    <limit lower="-1.91986218" upper="1.91986218" effort="107" velocity="3.142" />
+    <parent link="right_joint5" />
+    <child link="right_joint6" />
+    <axis xyz="0 0 1" />
+    <limit lower="-1.91986218" upper="1.91986218" effort="10" velocity="5" />
   </joint>
   <joint name="right_joint7" type="revolute">
     <origin xyz="-0.0993 0 -0.0615" rpy="0 -1.5707963 0" />
-    <parent link="right_link6" />
-    <child link="right_link7" />
-    <axis xyz="0 0 1" />
-    <limit lower="-3.14159265" upper="3.14159265" effort="36" velocity="3.142" />
+    <parent link="right_joint6" />
+    <child link="right_joint7" />
+    <axis xyz="0 0 1" />
+    <limit lower="-3.14159265" upper="3.14159265" effort="10" velocity="5" />
   </joint>
   <joint name="left_joint1" type="revolute">
     <origin xyz="0.32201385 -0.181 1.3500054" rpy="0 -1.3089969 3.1415927" />
     <parent link="left_arm_base" />
-    <child link="left_link1" />
-    <axis xyz="0 0 1" />
-    <limit lower="-3.14159265" upper="3.14159265" effort="647" velocity="1.309" />
+    <child link="left_joint1" />
+    <axis xyz="0 0 1" />
+    <limit lower="-3.14159265" upper="3.14159265" effort="10" velocity="5" />
   </joint>
   <joint name="left_joint2" type="revolute">
     <origin xyz="0.039999999 0 0.1512" rpy="0 -1.5707963 -3.1415927" />
-    <parent link="left_link1" />
-    <child link="left_link2" />
-    <axis xyz="0 0 1" />
-    <limit lower="-1.8325957145940461" upper="1.8325957145940461" effort="647" velocity="1.309" />
+    <parent link="left_joint1" />
+    <child link="left_joint2" />
+    <axis xyz="0 0 1" />
+    <limit lower="-1.8325957145940461" upper="1.8325957145940461" effort="10" velocity="5" />
   </joint>
   <joint name="left_joint3" type="revolute">
     <origin xyz="0.1795 0 -0.040000001" rpy="0 -1.5707963 3.1415927" />
-    <parent link="left_link2" />
-    <child link="left_link3" />
-    <axis xyz="0 0 1" />
-    <limit lower="-3.14159265" upper="3.14159265" effort="484" velocity="1.309" />
+    <parent link="left_joint2" />
+    <child link="left_joint3" />
+    <axis xyz="0 0 1" />
+    <limit lower="-3.14159265" upper="3.14159265" effort="10" velocity="5" />
   </joint>
   <joint name="left_joint4" type="revolute">
     <origin xyz="-1.2261866e-09 -0.068 0.3265" rpy="1.5707963 -1.3089969 -3.1415927" />
-    <parent link="left_link3" />
-    <child link="left_link4" />
-    <axis xyz="0 0 1" />
-    <limit lower="-2.53072742" upper="2.53072742" effort="459" velocity="1.749" />
+    <parent link="left_joint3" />
+    <child link="left_joint4" />
+    <axis xyz="0 0 1" />
+    <limit lower="-2.53072742" upper="2.53072742" effort="10" velocity="5" />
   </joint>
   <joint name="left_joint5" type="revolute">
     <origin xyz="0.22457775 0.060175428 0.068" rpy="1.5707963 0 1.8325957" />
-    <parent link="left_link4" />
-    <child link="left_link5" />
-    <axis xyz="0 0 1" />
-    <limit lower="-3.14159265" upper="3.14159265" effort="217" velocity="2.618" />
+    <parent link="left_joint4" />
+    <child link="left_joint5" />
+    <axis xyz="0 0 1" />
+    <limit lower="-3.14159265" upper="3.14159265" effort="10" velocity="5" />
   </joint>
   <joint name="left_joint6" type="revolute">
     <origin xyz="0.061499999 0 0.2415" rpy="0 -1.5707963 -3.1415927" />
-    <parent link="left_link5" />
-    <child link="left_link6" />
-    <axis xyz="0 0 1" />
-    <limit lower="-1.91986218" upper="1.91986218" effort="107" velocity="3.142" />
+    <parent link="left_joint5" />
+    <child link="left_joint6" />
+    <axis xyz="0 0 1" />
+    <limit lower="-1.91986218" upper="1.91986218" effort="10" velocity="5" />
   </joint>
   <joint name="left_joint7" type="revolute">
     <origin xyz="0.0993 0 -0.0615" rpy="0 -1.5707963 3.1415927" />
-    <parent link="left_link6" />
-    <child link="left_link7" />
-    <axis xyz="0 0 1" />
-    <limit lower="-3.14159265" upper="3.14159265" effort="36" velocity="3.142" />
+    <parent link="left_joint6" />
+    <child link="left_joint7" />
+    <axis xyz="0 0 1" />
+    <limit lower="-3.14159265" upper="3.14159265" effort="10" velocity="5" />
   </joint>
   <link name="right_arm_base" />
@@ -638,5 +638,5 @@
   <link name="right_tool0" />
   <joint name="right_tool0_fixed" type="fixed">
-    <parent link="right_link7" />
+    <parent link="right_joint7" />
     <child link="right_tool0" />
     <origin xyz="0 0 0.13585" rpy="0 0 0" />
@@ -649,5 +649,5 @@
   <link name="left_tool0" />
   <joint name="left_tool0_fixed" type="fixed">
-    <parent link="left_link7" />
+    <parent link="left_joint7" />
     <child link="left_tool0" />
     <origin xyz="0 0 0.13585" rpy="0 0 0" />

File: ros2_ws/src/alfa_robot_description/urdf/alfa_robot/robot_v3_end_effectors.xacro (robot description, xacro)
@@ -2,5 +2,5 @@
 <robot xmlns:xacro="http://wiki.ros.org/xacro" name="robot_v3_end_effectors">
   <xacro:macro name="v3_gripper" params="side">
-    <link name="${side}_link7">
+    <link name="${side}_joint7">
       <inertial>
         <origin xyz="-0.007153 0.051039 0.078079" rpy="0 0 0" />
@@ -48,5 +48,5 @@
     <joint name="${side}_moving_jaw_joint" type="prismatic">
       <origin xyz="0 0 0" rpy="0 0 0" />
-      <parent link="${side}_link7" />
+      <parent link="${side}_joint7" />
       <child link="${side}_moving_jaw" />
       <axis xyz="1 0 0" />
@@ -56,5 +56,5 @@
   </xacro:macro>
   <xacro:macro name="v3_suction" params="side">
-    <link name="${side}_link7">
+    <link name="${side}_joint7">
       <inertial>
         <origin xyz="-0.000330 -0.000125 0.070303" rpy="0 0 0" />
@@ -79,3 +79,28 @@
     </link>
   </xacro:macro>
+  <!-- Explicit golden scoop alias: identical V3.1.1 suction mechanics, verified upstream meshes. -->
+  <xacro:macro name="v3_scoop" params="side">
+    <link name="${side}_joint7">
+      <inertial>
+        <origin xyz="-0.000330 -0.000125 0.070303" rpy="0 0 0" />
+        <mass value="2.618" />
+        <inertia ixx="0.008369176" ixy="-0.000035407" ixz="-0.000011217" iyy="0.025870483" iyz="0.000004429" izz="0.027959973" />
+      </inertial>
+      <visual>
+        <material name="robot_v3_gray">
+          <color rgba="0.82 0.82 0.82 1" />
+        </material>
+        <origin xyz="0 0 0" rpy="0 0 0" />
+        <geometry>
+          <mesh filename="package://alfa_robot_description/meshes/robot_v3_scoop/scoop_visual.stl" scale="0.001 0.001 0.001" />
+        </geometry>
+      </visual>
+      <collision>
+        <origin xyz="-0.158443333 -0.088374996 0" rpy="0 0 0" />
+        <geometry>
+          <mesh filename="package://alfa_robot_description/meshes/robot_v3_scoop/scoop_collision.stl" scale="0.001 0.001 0.001" />
+        </geometry>
+      </collision>
+    </link>
+  </xacro:macro>
 </robot>
