Commit message: feat(curobo): 按旧范围换算双臂J2非对称限位并迁移规划资产

File: research/curobo_v3/generated/zero_model_candidate_20261018/mobile/robot_rezero_candidate.urdf (robot description, URDF)
Before this commit: robot alfa_robot_v3, 24 links, 23 joints
Joints:
- joint left_joint2: limit lower=-1.5707963267948966 upper=1.5707963267948966 effort=647 velocity=1.309 -> lower=-1.5707963267948966 upper=2.0943951023931953 effort=647 velocity=1.309
- joint right_joint2: limit lower=-1.5707963267948966 upper=1.5707963267948966 effort=647 velocity=1.309 -> lower=-2.0943951023931953 upper=1.5707963267948966 effort=647 velocity=1.309

File: research/curobo_v3/generated/zero_model_candidate_20261018/robot_rezero_candidate.urdf (robot description, URDF)
Before this commit: robot alfa_robot_v3, 21 links, 20 joints
Joints:
- joint left_joint2: limit lower=-1.5707963267948966 upper=1.5707963267948966 effort=647 velocity=1.309 -> lower=-1.5707963267948966 upper=2.0943951023931953 effort=647 velocity=1.309
- joint right_joint2: limit lower=-1.5707963267948966 upper=1.5707963267948966 effort=647 velocity=1.309 -> lower=-2.0943951023931953 upper=1.5707963267948966 effort=647 velocity=1.309

Commit message: feat(curobo): 反转J6方向并接入用户确认的新Home完整回归

File: research/curobo_v3/generated/zero_model_candidate_20261018/mobile/robot_rezero_candidate.urdf (robot description, URDF)
Before this commit: robot alfa_robot_v3, 24 links, 23 joints
Joints:
- joint left_joint6: axis 0 0 1 -> -0 -0 -1
- joint right_joint6: axis 0 0 1 -> -0 -0 -1

File: research/curobo_v3/generated/zero_model_candidate_20261018/robot_rezero_candidate.urdf (robot description, URDF)
Before this commit: robot alfa_robot_v3, 21 links, 20 joints
Joints:
- joint left_joint6: axis 0 0 1 -> -0 -0 -1
- joint right_joint6: axis 0 0 1 -> -0 -0 -1

Commit message: feat(curobo): 同步电控左J5新零位并更新URDF IK与Viser版本门禁

File: research/curobo_v3/generated/zero_model_candidate_20261018/mobile/robot_rezero_candidate.urdf (robot description, URDF)
Before this commit: robot alfa_robot_v3, 24 links, 23 joints
Joints:
- joint left_joint5: origin xyz=0 -0.241 -0.085 rpy=-1.5707963009899999 -1.570134696690499e-16 -3.1415926535894658 -> xyz=0 -0.241 -0.085 rpy=1.5707963009899999 1.570134696690499e-16 3.2736427763354125e-13

File: research/curobo_v3/generated/zero_model_candidate_20261018/robot_rezero_candidate.urdf (robot description, URDF)
Before this commit: robot alfa_robot_v3, 21 links, 20 joints
Joints:
- joint left_joint5: origin xyz=0 -0.241 -0.085 rpy=-1.5707963009899999 -1.570134696690499e-16 -3.1415926535894658 -> xyz=0 -0.241 -0.085 rpy=1.5707963009899999 1.570134696690499e-16 3.2736427763354125e-13

Commit message: feat(curobo): 采用确认后的双臂零位J6正向及191毫米TCP并同步FKIK

File: research/curobo_v3/generated/zero_model_candidate_20261018/mobile/robot_rezero_candidate.urdf (robot description, URDF)
Before this commit: robot alfa_robot_v3, 24 links, 23 joints
Joints:
- joint left_joint4: limit lower=-2.53072742 upper=2.53072742 effort=459 velocity=1.749 -> lower=-2.5080381397240736 upper=2.553416700275926 effort=459 velocity=1.749; origin xyz=0 0.085000001 0.26 rpy=-1.5707963000000003 0 0 -> xyz=0 0.085000001 0.26 rpy=-1.5707962999931016 -0.022689280275926271 -6.0806126187813901e-10
- joint left_joint5: origin xyz=0 -0.241 -0.085 rpy=1.5707963009899999 1.570134696690499e-16 3.2736427763354125e-13 -> xyz=0 -0.241 -0.085 rpy=-1.5707963009899999 -3.1402271553742868e-16 -3.1415926535894658
- joint left_joint6: axis -0 -0 -1 -> 0 0 1
- joint left_tool0_fixed: origin xyz=0 0 0.151 rpy=0 0 0 -> xyz=0 0 0.191 rpy=0 0 0
- joint right_joint6: axis -0 -0 -1 -> 0 0 1
- joint right_tool0_fixed: origin xyz=0 0 0.151 rpy=0 0 0 -> xyz=0 0 0.191 rpy=0 0 0

File: research/curobo_v3/generated/zero_model_candidate_20261018/robot_rezero_candidate.urdf (robot description, URDF)
Before this commit: robot alfa_robot_v3, 21 links, 20 joints
Joints:
- joint left_joint4: limit lower=-2.53072742 upper=2.53072742 effort=459 velocity=1.749 -> lower=-2.5080381397240736 upper=2.553416700275926 effort=459 velocity=1.749; origin xyz=0 0.085000001 0.26 rpy=-1.5707963000000003 0 0 -> xyz=0 0.085000001 0.26 rpy=-1.5707962999931016 -0.022689280275926271 -6.0806126187813901e-10
- joint left_joint5: origin xyz=0 -0.241 -0.085 rpy=1.5707963009899999 1.570134696690499e-16 3.2736427763354125e-13 -> xyz=0 -0.241 -0.085 rpy=-1.5707963009899999 -3.1402271553742868e-16 -3.1415926535894658
- joint left_joint6: axis -0 -0 -1 -> 0 0 1
- joint left_tool0_fixed: origin xyz=0 0 0.151 rpy=0 0 0 -> xyz=0 0 0.191 rpy=0 0 0
- joint right_joint6: axis -0 -0 -1 -> 0 0 1
- joint right_tool0_fixed: origin xyz=0 0 0.151 rpy=0 0 0 -> xyz=0 0 0.191 rpy=0 0 0

Commit message: fix(curobo): 删除误加J4零位偏置与本地小角度拟合补偿

File: research/curobo_v3/generated/zero_model_candidate_20261018/mobile/robot_rezero_candidate.urdf (robot description, URDF)
Before this commit: robot alfa_robot_v3, 24 links, 23 joints
Joints:
- joint left_joint4: limit lower=-2.5080381397240736 upper=2.553416700275926 effort=459 velocity=1.749 -> lower=-2.53072742 upper=2.53072742 effort=459 velocity=1.749; origin xyz=0 0.085000001 0.26 rpy=-1.5707962999931016 -0.022689280275926271 -6.0806126187813901e-10 -> xyz=0 0.085000001 0.26 rpy=-1.5707963000000003 0 0
- joint left_joint5: origin xyz=0 -0.241 -0.085 rpy=-1.5707963009899999 -3.1402271553742868e-16 -3.1415926535894658 -> xyz=0 -0.241 -0.085 rpy=-1.5707963009899999 -1.570134696690499e-16 -3.1415926535894658

File: research/curobo_v3/generated/zero_model_candidate_20261018/robot_rezero_candidate.urdf (robot description, URDF)
Before this commit: robot alfa_robot_v3, 21 links, 20 joints
Joints:
- joint left_joint4: limit lower=-2.5080381397240736 upper=2.553416700275926 effort=459 velocity=1.749 -> lower=-2.53072742 upper=2.53072742 effort=459 velocity=1.749; origin xyz=0 0.085000001 0.26 rpy=-1.5707962999931016 -0.022689280275926271 -6.0806126187813901e-10 -> xyz=0 0.085000001 0.26 rpy=-1.5707963000000003 0 0
- joint left_joint5: origin xyz=0 -0.241 -0.085 rpy=-1.5707963009899999 -3.1402271553742868e-16 -3.1415926535894658 -> xyz=0 -0.241 -0.085 rpy=-1.5707963009899999 -1.570134696690499e-16 -3.1415926535894658
